File: Hardware/PCB/Muhammad_PCB_5.0.0/MothBox/MothBo.kicad_pcb (KiCad board)
At the start: 2 copper layers, 237 x 140.5 mm, 178 parts, among them J1 Screw_Terminal_01x02, J2 TYPE-C-31-M-17, J4 GPS Header, J5 Conn_01x05_Pin, J7 DC Power Jack, Q1 IRF9540N, Q10 BC817, Q11 BC817, Q2 TJ10S04M3L,LXHQ, Q3 BC817, Q4 TJ10S04M3L,LXHQ, Q5 TJ10S04M3L,LXHQ, Q6 BC817, Q7 BC817, Q8 BC817, Q9 BC817, SW1 SW_Push, SW2 Days, SW3 Power, SW4 Sequence+Toggle, SW5 Hours, SW6 Hours, U1 XL4015, U10 IRF9335TRPBF, U11 IRF9335TRPBF, U12 CD74HC4067M96E4, U13 CD74HC4067M96E4, U2 9V-36V to 12V 5A 60W, U3 RASPBERRY_PI_5, U4 RASPBERRY_PI_4B_4GB, U5 STM32L031K6Tx, U6 TLV75733PDBVR, U8 IRF9335TRPBF, U9 IRF9335TRPBF, Y1 32.768kHz

Commit message: changed mothbox version number
Other:
- board text added: "MOTHBOX V5.0.0"
Changed lines of the file:
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@@
 		)
 	)
-	(gr_text "MOTHBOX V4.5"
-		(at 161.1 160.915671 0)
+	(gr_text "MOTHBOX V5.0.0"
+		(at 159 160.915671 0)
 		(layer "F.SilkS" knockout)
 		(effects
