File: Hardware/PCB/Andy_PCB_5.0.0/MothBox/MothBo.kicad_pcb (KiCad board)
At the start: 2 copper layers, 237.2 x 140.5 mm, 179 parts, among them J1 Screw_Terminal_01x02, J2 TYPE-C-31-M-17, J4 GPS Header, J5 Conn_01x05_Pin, J7 DC Power Jack, Q1 IRF9540N, Q10 BC817, Q11 BC817, Q2 TJ10S04M3L,LXHQ, Q3 BC817, Q4 TJ10S04M3L,LXHQ, Q5 TJ10S04M3L,LXHQ, Q6 BC817, Q7 BC817, Q8 BC817, Q9 BC817, SW1 SW_Push, SW2 Days, SW3 Power, SW4 seq tog, SW5 Hours, SW6 Hours, U1 XL4015, U10 IRF9335TRPBF, U11 IRF9335TRPBF, U12 CD74HC4067M96E4, U13 CD74HC4067M96E4, U2 9V-36V to 12V 5A 60W, U3 RASPBERRY_PI_5, U4 RASPBERRY_PI_4B_4GB, U5 STM32L031K6Tx, U6 TLV75733PDBVR, U8 IRF9335TRPBF, U9 IRF9335TRPBF, Y1 32.768kHz

Commit message: Andy more tweaks
Parts:
- moved C6 104.7 mm to (116.6, 181.9), turned to 180 degrees
- moved C7 100.4 mm to (120.8, 177.5), turned to 180 degrees
- moved U6 100.3 mm to (116.8, 178.6), turned to 0 degrees
- moved D31 97.7 mm to (111.5, 181.1), turned to 0 degrees
- moved C9 95.7 mm to (120.8, 174.1), turned to 180 degrees
- moved R11 94.9 mm to (117.5, 174.5), turned to -90 degrees
- moved C10 93.1 mm to (126.7, 169.8), turned to 180 degrees
- moved C15 92.9 mm to (120.8, 172.0), turned to 180 degrees
- moved D9 90.6 mm to (68.5, 169.8), turned to 0 degrees
- moved C11 89.8 mm to (126.7, 167.2), turned to 180 degrees
- moved Y1 89.7 mm to (123.7, 168.5), turned to 90 degrees
- moved R82 89.5 mm to (107.5, 180.2), turned to 90 degrees
- moved U11 88.0 mm to (107.5, 174.1), turned to 0 degrees
- moved R63 84.2 mm to (78.7, 170.4), turned to 180 degrees
- moved U5 83.9 mm to (115.5, 166.9), turned to 180 degrees
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Routing:
- net /UV LED PCB/+12V_PCB3: vias 4 -> 0
- net /UV LED PCB/+12V_PCB2: vias 4 -> 0
- net /UV LED PCB/+12V_PCB1: vias 4 -> 0
- net +12V: vias 12 -> 0
