File: Hardware/PCB/Andy_PCB_5.0.0/MothBox/GPS.kicad_sch (KiCad schematic)
At the start: 10 parts, among them U1 Days, U17 GPs 5 pin PM2.54-1*5, U2 Hours1, U6 Hours2, U7 Modes, U8 CD74HC4067M96E4, U9 CD74HC4067M96E4

Commit message: Maybe these files needed saving too for paul?
Parts:
- C16, C17: symbol Device:C_Small -> MB_Library:C_Small
- H9: symbol easyeda2kicad:2.54-1*4P母 -> MB_Library:2.54-1*4P母
- U1, U2, U6, U7: symbol easyeda2kicad:SMXS-08K-TP -> MB_Library:SMXS-08K-TP
- U17: symbol easyeda2kicad:PM2.54-1*5 -> MB_Library:PM2.54-1*5
- U8: symbol CD74HC4067M96E4:CD74HC4067M96E4 -> MB_Library:CD74HC4067M96E4_1
- U9: symbol CD74HC4067M96E4:CD74HC4067M96E4 -> MB_Library:CD74HC4067M96E4
Changed lines of the file:
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@@
 	)
 	(symbol
-		(lib_id "power:+3.3V")
+		(lib_id "MB_Library:+3.3V")
 		(at 33.02 64.77 90)
 		(unit 1)
@@
 	)
 	(symbol
-		(lib_id "easyeda2kicad:2.54-1*4P母")
+		(lib_id "MB_Library:2.54-1*4P母")
 		(at 38.1 45.72 0)
 		(unit 1)
@@
 	)
 	(symbol
-		(lib_id "power:GND")
+		(lib_id "MB_Library:GND")
 		(at 227.33 100.33 0)
 		(unit 1)
@@
 	)
 	(symbol
-		(lib_id "power:GND")
+		(lib_id "MB_Library:GND")
 		(at 181.61 96.52 0)
 		(unit 1)
@@
 	)
 	(symbol
-		(lib_id "power:+3.3V")
+		(lib_id "MB_Library:+3.3V")
 		(at 33.02 41.91 90)
 		(unit 1)
@@
 	(symbol
 		(lib_name "CD74HC4067M96E4_1")
-		(lib_id "CD74HC4067M96E4:CD74HC4067M96E4")
+		(lib_id "MB_Library:CD74HC4067M96E4_1")
 		(at 100.33 153.67 0)
 		(unit 1)
@@
 	)
 	(symbol
-		(lib_id "power:GND")
+		(lib_id "MB_Library:GND")
 		(at 33.02 67.31 270)
 		(unit 1)
@@
 	)
 	(symbol
-		(lib_id "Device:C_Small")
+		(lib_id "MB_Library:C_Small")
 		(at 125.73 133.35 180)
 		(unit 1)
@@
 	)
 	(symbol
-		(lib_id "power:GND")
+		(lib_id "MB_Library:GND")
 		(at 125.73 135.89 0)
 		(unit 1)
@@
 	)
 	(symbol
-		(lib_id "power:GND")
+		(lib_id "MB_Library:GND")
 		(at 123.19 173.99 0)
 		(unit 1)
@@
 	)
 	(symbol
-		(lib_id "easyeda2kicad:SMXS-08K-TP")
+		(lib_id "MB_Library:SMXS-08K-TP")
 		(at 273.05 82.55 0)
 		(unit 1)
@@
 	)
 	(symbol
-		(lib_id "easyeda2kicad:PM2.54-1*5")
+		(lib_id "MB_Library:PM2.54-1*5")
 		(at 38.1 69.85 0)
 		(unit 1)
@@
 	)
 	(symbol
-		(lib_id "power:GND")
+		(lib_id "MB_Library:GND")
 		(at 231.14 175.26 0)
 		(unit 1)
@@
 	)
 	(symbol
-		(lib_id "easyeda2kicad:SMXS-08K-TP")
+		(lib_id "MB_Library:SMXS-08K-TP")
 		(at 181.61 78.74 0)
 		(unit 1)
@@
 	)
 	(symbol
-		(lib_id "power:+3.3V")
+		(lib_id "MB_Library:+3.3V")
 		(at 125.73 124.46 0)
 		(unit 1)
@@
 	)
 	(symbol
-		(lib_id "easyeda2kicad:SMXS-08K-TP")
+		(lib_id "MB_Library:SMXS-08K-TP")
 		(at 237.49 82.55 0)
 		(unit 1)
@@
 	)
 	(symbol
-		(lib_id "power:GND")
+		(lib_id "MB_Library:GND")
 		(at 236.22 135.89 0)
 		(unit 1)
@@
 	)
 	(symbol
-		(lib_id "power:+3.3V")
+		(lib_id "MB_Library:+3.3V")
 		(at 236.22 124.46 0)
 		(unit 1)
@@
 	)
 	(symbol
-		(lib_id "easyeda2kicad:SMXS-08K-TP")
+		(lib_id "MB_Library:SMXS-08K-TP")
 		(at 130.81 78.74 0)
 		(unit 1)
@@
 	)
 	(symbol
-		(lib_id "power:GND")
+		(lib_id "MB_Library:GND")
 		(at 262.89 100.33 0)
 		(unit 1)
@@
 	)
 	(symbol
-		(lib_id "Device:C_Small")
+		(lib_id "MB_Library:C_Small")
 		(at 236.22 133.35 180)
 		(unit 1)
@@
 	)
 	(symbol
-		(lib_id "power:GND")
+		(lib_id "MB_Library:GND")
 		(at 33.02 49.53 0)
 		(unit 1)
@@
 	)
 	(symbol
-		(lib_id "power:GND")
+		(lib_id "MB_Library:GND")
 		(at 123.19 97.79 0)
 		(unit 1)
@@
 	)
 	(symbol
-		(lib_id "CD74HC4067M96E4:CD74HC4067M96E4")
+		(lib_id "MB_Library:CD74HC4067M96E4")
 		(at 210.82 153.67 0)
 		(unit 1)
