File: Hardware/PCB/Andy_PCB_5.0.0/MothBoxSeeed/MothBo.kicad_pcb (KiCad board)
At the start: 2 copper layers, 237.2 x 140.5 mm, 179 parts, among them J1 Screw_Terminal_01x02, J2 TYPE-C-31-M-17, J4 GPS Header, J5 Conn_01x05_Pin, J7 DC Power Jack, Q1 IRF9540N, Q10 BC817, Q11 BC817, Q2 TJ10S04M3L,LXHQ, Q3 BC817, Q4 TJ10S04M3L,LXHQ, Q5 TJ10S04M3L,LXHQ, Q6 BC817, Q7 BC817, Q8 BC817, Q9 BC817, SW1 SW_Push, SW2 Days, SW3 Power, SW4 seq tog, SW5 Hours, SW6 Hours, U1 XL4015, U10 IRF9335TRPBF, U11 IRF9335TRPBF, U12 CD74HC4067M96E4, U13 CD74HC4067M96E4, U2 9V-36V to 12V 5A 60W, U3 RASPBERRY_PI_5, U4 RASPBERRY_PI_4B_4GB, U5 STM32L031K6Tx, U6 TLV75733PDBVR, U8 IRF9335TRPBF, U9 IRF9335TRPBF, Y1 32.768kHz

Commit message: first JLCPCB build
Parts:
- SW4: value seq tog -> Sequence+Toggle
Routing:
- net /RPI5+MCU/NRST: track 178.8 -> 192.6 mm
- net /RPI5+MCU/SWDIO: track 187.7 -> 197.6 mm, vias 1 -> 2
- net /RPI5+MCU/SWDCLK: track 199.4 -> 200.2 mm, vias 1 -> 2
- net GND: vias 382 -> 381
Other:
- outline, holes or cut-outs redrawn
