File: Hardware/PCB/Andy_PCB_5.0.1/MothBox/Photo LEDS's.kicad_sch (KiCad schematic)
At the start: 76 parts, among them Q3 BC817, Q4 SUD50P06-15-GE3, Q5 BC817, Q6 SUD50P06-15-GE3

Commit message: daily schematic updates
Parts:
- removed Q3, Q5: BC817, Package_TO_SOT_SMD:SOT-23, symbol MB_Library:BC817_NPN_BJT
- removed Q4, Q6: SUD50P06-15-GE3, easyeda2kicad:TO-252-3_L6.5-W5.8-P4.58-BL, symbol MB_Library:SUD50P06-15-GE3
- removed R19: 1k, Resistor_SMD:R_0805_2012Metric, symbol MB_Library:R_US
- removed R21: 10k, Resistor_SMD:R_0805_2012Metric, symbol MB_Library:R_US
- removed TP5: LEDCTRL_R, TestPoint:TestPoint_THTPad_D1.0mm_Drill0.5mm, symbol MB_Library:TestPoint
- added Q12, Q3: YJQ10N2A, Pauls_Footprints:DFN2020-3, symbol _pauls_library:YJQ10N2A
- R17: value FRC0805F30R0TS -> 30R
- R9: value 1k -> 10k; LCSC Part no  C95781 -> C84376
- TP3: value LEDCTRL_L -> LEDCTRL
Connections:
- net +12V: now also R10.2, R12.2, R13.2, R14.2, R15.2, R16.2, R17.2, R18.2, R20.2, R22.2, R23.2, R24.2, R25.2, R26.2, R7.2, R8.2; no longer R11.2
- net GND: now also R11.1, R9.1, Q12.4 (S), Q12.7 (S), Q3.4 (S), Q3.7 (S); no longer LED12.1 (K), LED15.1 (K), LED18.1 (K), LED21.1 (K), LED24.1 (K), LED27.1 (K), LED3.1 (K), LED30.1 (K), LED33.1 (K), LED36.1 (K), LED39.1 (K), LED42.1 (K), LED45.1 (K), LED48.1 (K), LED6.1 (K), LED9.1 (K)
- removed net +12V_L_LED: R10.2, R12.2, R13.2, R14.2, R15.2, R16.2, R7.2, R8.2, TP4.1
- removed net +12V_R_LED: R17.2, R18.2, R20.2, R22.2, R23.2, R24.2, R25.2, R26.2, TP6.1
- net L_LED_CTRL renamed PHOTO_LED_CTRL
- net PHOTO_LED_CTRL: now also R11.2, Q12.3 (D), Q3.3 (D)
- new net: LED27.1 (K), LED30.1 (K), LED33.1 (K), LED36.1 (K), LED39.1 (K), LED42.1 (K), LED45.1 (K), LED48.1 (K), Q3.1 (D), Q3.2 (D), Q3.3 (D), Q3.5 (D), Q3.6 (D), Q3.8 (D), TP6.1
- new net: LED12.1 (K), LED15.1 (K), LED18.1 (K), LED21.1 (K), LED24.1 (K), LED3.1 (K), LED6.1 (K), LED9.1 (K), Q12.1 (D), Q12.2 (D), Q12.3 (D), Q12.5 (D), Q12.6 (D), Q12.8 (D), TP4.1
Other:
- note added: "30R"
- note added: "PH: Measure the current flowing through the LED strings. Does the resistance need to be modified?"
- moved on the sheet: LED1, LED10, LED11, LED12, LED13, LED14, LED15, LED16, LED17, LED18, LED19, LED2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
