File: Hardware/PCB/Andy_PCB_5.0.1/MothBox/MothBox.kicad_pcb (KiCad board)
At the start: 2 copper layers, 237 x 140.5 mm, 147 parts, among them P1 Raw Input, P2 12V Regulated Input, P3 Input to regulator, P4 External Attractor, Q1 BC817, Q10 BC817, Q11 BC817, Q2 SUD50P06-15-GE3, Q4 BC817, Q5 SUD50P06-15-GE3, Q6 BC817, Q7 SUD50P06-15-GE3, Q8 BC817, Q9 BC817, U1 Days, U10 FDS4435BZ, U11 FDS4435BZ, U12 FDS4435BZ, U13 FDS4435BZ, U16 Female Inv Socket Pi 2.54-2*20, U17 GPs 5 pin PM2.54-1*5, U18 RASPBERRY_PI_4B_4GB, U19 INA219BIDCNT, U2 Hours1, U3 XL4015E1, U5 RASPBERRY_PI_5, U6 Hours2, U7 Modes, U8 CD74HC4067M96E4, U9 CD74HC4067M96E4

Commit message: updated photo LEDs and the power page
Parts:
- removed A1, A2, A3: PZ254R-11-04P, MB_Library:HDR-TH_4P-P2.54-H-M-W10.4
- removed C17: 0.1uF, MB_Library:C_0805_2012Metric
- removed D30, D32, D33: ESD12VD3B-TP, MB_Library:D_SOD-323
- removed Q10, Q11, Q4, Q6, Q8, Q9: BC817, MB_Library:SOT-23
- removed Q5, Q7: SUD50P06-15-GE3, MB_Library:TO-252-3_L6.5-W5.8-P4.58-BL
- removed R54, R66, R75, R76, R79, R80: 1k, MB_Library:R_0805_2012Metric
- removed R57, R69, R77, R78, R81, R82: 10k, MB_Library:R_0805_2012Metric
- removed the TP1 at (252.0, 201.3)
- removed the TP2 at (248.5, 198.8)
- removed TP8: LEDCTRL_R, MB_Library:TestPoint_THTPad_D1.0mm_Drill0.5mm
- removed the U10 at (255.5, 94.3)
- removed the U11 at (206.0, 67.8)
- removed U12: FDS4435BZ, MB_Library:SOIC-8_L5.0-W4.0-P1.27-LS6.0-BL
- removed the U13 at (254.1, 129.6)
- removed the U8 at (170.5, 90.3)
- removed U9: CD74HC4067M96E4, MB_Library:SOIC-24_L15.4-W7.5-P1.27-LS10.3-BL
- added C9: 0.1uF, Capacitor_SMD:C_0805_2012Metric, F.Cu at (317.6, 123.6)
- added D5: ESD12VD3B-TP, Diode_SMD:D_SOD-323, F.Cu at (321.9, 128.5)
- added D6: ESD12VD3B-TP, Diode_SMD:D_SOD-323, F.Cu at (321.9, 131.5)
- added D7: ESD12VD3B-TP, Diode_SMD:D_SOD-323, F.Cu at (321.9, 134.4)
- added R11: 10k, Resistor_SMD:R_0805_2012Metric, F.Cu at (328.2, 131.5)
- added R19: 10k, Resistor_SMD:R_0805_2012Metric, F.Cu at (317.5, 128.5)
- added R21: 10k, Resistor_SMD:R_0805_2012Metric, F.Cu at (317.5, 131.5)
- added R27: 10k, Resistor_SMD:R_0805_2012Metric, F.Cu at (317.5, 134.4)
- added R28: 10k, Resistor_SMD:R_0805_2012Metric, F.Cu at (317.5, 137.4)
- added R9: 10k, Resistor_SMD:R_0805_2012Metric, F.Cu at (328.2, 128.5)
- added U15: PCA9535PW, Package_SO:TSSOP-24_4.4x7.8mm_P0.65mm, F.Cu at (320.1, 117.4)
- added U16: PCA9535PW, Package_SO:TSSOP-24_4.4x7.8mm_P0.65mm, F.Cu at (329.2, 117.4)
- B1: footprint MB_Library:Talentcell -> AQLibrary:Talentcell
- C1: footprint MB_Library:CP_Elec_10x12.5 -> Capacitor_SMD:CP_Elec_10x12.5
- C2, C3, C5: footprint MB_Library:C_0805_2012Metric_Pad1.18x1.45mm_HandSolder -> Capacitor_SMD:C_0805_2012Metric_Pad1.18x1.45mm_HandSolder
- C4: footprint MB_Library:CP_Elec_10x10 -> Capacitor_SMD:CP_Elec_10x10
- C6: value 0.1µF -> 0.1uF; footprint MB_Library:C0603 -> Capacitor_SMD:C_0603_1608Metric; moved to F.Cu
- C7: renamed from C16; footprint MB_Library:C_0805_2012Metric -> Capacitor_SMD:C_0805_2012Metric
- D2: renamed from D31; footprint MB_Library:D_SOD-323 -> Diode_SMD:D_SOD-323
- F1: renamed from F2; value Polyfuse -> 5A
- H1: renamed from H9; footprint MB_Library:GPS4pin_HDR-TH_4P-P2.54-V-F -> AQLibrary:GPS4pin_HDR-TH_4P-P2.54-V-F
- H2: renamed from H3; footprint MB_Library:MountingHole_6.4mm_M6_Pad -> MountingHole:MountingHole_6.4mm_M6_Pad
- H3: renamed from H2; footprint MB_Library:MountingHole_6.4mm_M6_Pad -> MountingHole:MountingHole_6.4mm_M6_Pad
- H4: renamed from H1; footprint MB_Library:MountingHole_6.4mm_M6_Pad -> MountingHole:MountingHole_6.4mm_M6_Pad
- H5: renamed from H8; footprint MB_Library:MountingHole_6.4mm_M6_Pad -> MountingHole:MountingHole_6.4mm_M6_Pad
- H6: footprint MB_Library:MountingHole_6.4mm_M6_Pad -> MountingHole:MountingHole_6.4mm_M6_Pad
- H7: renamed from H5; footprint MB_Library:MountingHole_6.4mm_M6_Pad -> MountingHole:MountingHole_6.4mm_M6_Pad
- L1: footprint MB_Library:L_Chilisin_BMRG00131360 -> Inductor_SMD:L_Chilisin_BMRG00131360
- Q1: footprint MB_Library:SOT-23 -> Package_TO_SOT_SMD:SOT-23
- R1: footprint MB_Library:R_0805_2012Metric -> Resistor_SMD:R_0805_2012Metric
- R17: renamed from R10; value FRC0805F30R0TS -> 30R
- R2: renamed from R4; footprint MB_Library:C_0805_2012Metric_Pad1.18x1.45mm_HandSolder -> Capacitor_SMD:C_0805_2012Metric_Pad1.18x1.45mm_HandSolder
- R3: renamed from R5; footprint MB_Library:C_0805_2012Metric_Pad1.18x1.45mm_HandSolder -> Capacitor_SMD:C_0805_2012Metric_Pad1.18x1.45mm_HandSolder
- R4: renamed from R63; value 0.1/1% (PT2512FK-070R1L) -> 0.1R/1% (PT2512FK-070R1L)
- R5: renamed from R64; value 10k -> 4.7K
- R6: renamed from R65; value 10k -> 4.7K
- TP1: renamed from TP3; footprint MB_Library:TestPoint_THTPad_D1.0mm_Drill0.5mm -> TestPoint:TestPoint_THTPad_D1.0mm_Drill0.5mm
- TP2: renamed from TP4; footprint MB_Library:TestPoint_THTPad_D1.0mm_Drill0.5mm -> TestPoint:TestPoint_THTPad_D1.0mm_Drill0.5mm
- TP3: renamed from TP7; value LEDCTRL_L -> LEDCTRL; footprint MB_Library:TestPoint_THTPad_D1.0mm_Drill0.5mm -> TestPoint:TestPoint_THTPad_D1.0mm_Drill0.5mm
- TP4: renamed from TP5; footprint MB_Library:TestPoint_THTPad_D1.0mm_Drill0.5mm -> TestPoint:TestPoint_THTPad_D1.0mm_Drill0.5mm
- TP6: footprint MB_Library:TestPoint_THTPad_D1.0mm_Drill0.5mm -> TestPoint:TestPoint_THTPad_D1.0mm_Drill0.5mm
- U19: renamed from U14; footprint MB_Library:Arducam Owlsight -> Attractor:Arducam Owlsight
- U5: footprint MB_Library:EPAPER_PinHeader_2x20_P2.54mm_Vertical -> AQLibrary:EPAPER_PinHeader_2x20_P2.54mm_Vertical
- U6: renamed from U18; footprint MB_Library:MODULE_RASPBERRY_PI_4B_4GB_Sideways -> RASPBERRY_PI_4B_4GB:MODULE_RASPBERRY_PI_4B_4GB_Sideways
- U8: renamed from U17; footprint MB_Library:GPS5pin_HDR-TH_5P-P2.54-V-F -> AQLibrary:GPS5pin_HDR-TH_5P-P2.54-V-F
- moved C6 86.9 mm to (328.0, 136.2), turned to 0 degrees
- renumbered E3 to E1, LED12 to LED1, LED9 to LED10, LED10 to LED11, LED11 to LED12, LED1 to LED2, LED34 to LED20, LED35 to LED21, LED47 to LED22, LED48 to LED23, LED49 to LED24, LED20 to LED25, LED21 to LED26, LED22 to LED27, LED23 to LED28, LED24 to LED29, LED2 to LED3, LED25 to LED30, LED26 to LED31, LED27 to LED32, LED28 to LED33, LED29 to LED34, LED36 to LED35, LED37 to LED36, LED38 to LED37, LED39 to LED38, LED40 to LED39, LED3 to LED4, LED41 to LED40, LED42 to LED41, LED43 to LED42, LED44 to LED43, LED45 to LED44, LED46 to LED45, LED50 to LED46, LED51 to LED47, LED52 to LED48, LED4 to LED5, LED5 to LED6, LED6 to LED7, LED7 to LED8, LED8 to LED9, P3 to P2, P2 to P3, R3 to R10, R6 to R12, R7 to R13, R8 to R14, R9 to R15, R53 to R16, R11 to R18, R12 to R20, R13 to R22, R14 to R23, R15 to R24, R52 to R25, R55 to R26, R51 to R7, R2 to R8, U1 to U10, U7 to U11, U2 to U13, U6 to U14, U3 to U2, U19 to U3, U16 to U7
Connections:
- net /Power/FB renamed Net-(U2-FB)
- net L_LED_CTRL renamed PHOTO_LED_CTRL
- C6 pad 1: GND -> +3.3V
- C6 pad 2: +3.3V -> GND
- D2 pad 1: /UV LED PCB/+12V_PCB2 -> +12V
- E1 pad 1: Net-(E3-C) -> Net-(E1-C)
- L1 pad 1: Net-(E3-C) -> Net-(E1-C)
- LED12 pad 1: GND -> Net-(LED12-K)
- LED15 pad 1: GND -> Net-(LED12-K)
- LED18 pad 1: GND -> Net-(LED12-K)
- LED21 pad 1: GND -> Net-(LED12-K)
- LED24 pad 1: GND -> Net-(LED12-K)
- LED27 pad 1: GND -> Net-(LED27-K)
- LED3 pad 1: GND -> Net-(LED12-K)
- LED30 pad 1: GND -> Net-(LED27-K)
- LED33 pad 1: GND -> Net-(LED27-K)
- LED36 pad 1: GND -> Net-(LED27-K)
- LED39 pad 1: GND -> Net-(LED27-K)
- LED42 pad 1: GND -> Net-(LED27-K)
- LED45 pad 1: GND -> Net-(LED27-K)
- LED48 pad 1: GND -> Net-(LED27-K)
- LED6 pad 1: GND -> Net-(LED12-K)
- LED9 pad 1: GND -> Net-(LED12-K)
- P4 pad 1: GND -> Net-(P4-Pad1)
- P4 pad 2: /UV LED PCB/+12V_PCB4 -> +12V
- R10 pad 2: /Photo LED's/+12V_L_LED -> +12V
- R12 pad 2: /Photo LED's/+12V_L_LED -> +12V
- R13 pad 2: /Photo LED's/+12V_L_LED -> +12V
- R14 pad 2: /Photo LED's/+12V_L_LED -> +12V
- R15 pad 2: /Photo LED's/+12V_L_LED -> +12V
- R16 pad 2: /Photo LED's/+12V_L_LED -> +12V
- R17 pad 2: /Photo LED's/+12V_R_LED -> +12V
- R18 pad 2: /Photo LED's/+12V_R_LED -> +12V
- R20 pad 2: /Photo LED's/+12V_R_LED -> +12V
- R22 pad 2: /Photo LED's/+12V_R_LED -> +12V
- R23 pad 2: /Photo LED's/+12V_R_LED -> +12V
- R24 pad 2: /Photo LED's/+12V_R_LED -> +12V
- R25 pad 2: /Photo LED's/+12V_R_LED -> +12V
- R26 pad 2: /Photo LED's/+12V_R_LED -> +12V
- R4 pad 1: /Power/VIN- -> /Power/VIN+
- R4 pad 2: /Power/VIN+ -> /Power/VIN-
- R7 pad 2: /Photo LED's/+12V_L_LED -> +12V
- R8 pad 2: /Photo LED's/+12V_L_LED -> +12V
- TP2 pad 1: /Power/VIN- -> unconnected-(TP2-Pad1)
- TP4 pad 1: /Photo LED's/+12V_L_LED -> Net-(LED12-K)
- TP6 pad 1: /Photo LED's/+12V_R_LED -> Net-(LED27-K)
- U2 pad 3: Net-(E3-C) -> Net-(E1-C)
- U2 pad 6: unconnected-(U3-SW-Pad6) -> Net-(E1-C)
- U3 pad 7: Net-(U19-A0) -> GND
- U3 pad 8: Net-(U19-A1) -> GND
- U5 pad 17: unconnected-(U5-3V3-Pad17) -> +3.3V
- U7 pad 11: S2_MUX -> unconnected-(U7-Pad11)
- U7 pad 14: S1_MUX -> unconnected-(U7-Pad14)
- U7 pad 16: S3_MUX -> unconnected-(U7-Pad16)
- U7 pad 30: EN_MUX1 -> UV2_CTRL
- U7 pad 32: EN_MUX2 -> UV3_CTRL
- U7 pad 34: S0_MUX -> unconnected-(U7-Pad34)
- U7 pad 35: COM_I/O -> unconnected-(U7-Pad35)
Routing:
- net unconnected-(U7-Pad34): track 0.00 -> 193.6 mm, vias 0 -> 6
- net S0_MUX: track 193.6 -> 0.00 mm, vias 6 -> 0
- net unconnected-(U7-Pad14): track 0.00 -> 181.7 mm, vias 0 -> 8
- net S1_MUX: track 181.7 -> 0.00 mm, vias 8 -> 0
- net unconnected-(U7-Pad16): track 0.00 -> 180.6 mm, vias 0 -> 2
- net S3_MUX: track 180.6 -> 0.00 mm, vias 2 -> 0
- net unconnected-(U7-Pad11): track 0.00 -> 165.9 mm, vias 0 -> 4
- net S2_MUX: track 165.9 -> 0.00 mm, vias 4 -> 0
- net unconnected-(U7-Pad35): track 0.00 -> 148.5 mm, vias 0 -> 3
- net COM_I/O: track 148.5 -> 0.00 mm, vias 3 -> 0
- net UV3_CTRL: track 0.00 -> 141.7 mm, vias 0 -> 4
- net EN_MUX2: track 141.7 -> 0.00 mm, vias 4 -> 0
- net (no net): track 0.00 -> 126.3 mm, vias 0 -> 1
- net UV2_CTRL: track 0.00 -> 79.3 mm
- net EN_MUX1: track 79.3 -> 0.00 mm
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
Commit message: updated footprints and schematic
Parts:
- removed F1: 5A, MB_Library:F0805
- removed P1: Raw Input, MB_Library:CONN-TH_2P-P5.08_DIBO_DB142R-5.08-2P
- removed P2: Input to regulator, MB_Library:CONN-TH_2P-P5.08_DIBO_DB142R-5.08-2P
- removed P3: 12V Regulated Input, MB_Library:CONN-TH_2P-P5.08_DIBO_DB142R-5.08-2P
- removed P4: External Attractor, MB_Library:CONN-TH_2P-P5.08_DIBO_DB142R-5.08-2P
- removed R1: 10k, Resistor_SMD:R_0805_2012Metric
- removed TP2: VIN_-, TestPoint:TestPoint_THTPad_D1.0mm_Drill0.5mm
- added D1: 10V, Diode_SMD:D_SOD-323, F.Cu at (400.7, 158.4)
- added F2: 6A trip, Resistor_SMD:R_1812_4532Metric, F.Cu at (402.0, 149.8)
- added H10: PZ254R-12-8P, easyeda_footprints:HDR-TH_8P-P2.54-H-M-R2-C4-S2.54, F.Cu at (436.0, 135.4)
- added H8: PZ254R-12-8P, easyeda_footprints:HDR-TH_8P-P2.54-H-M-R2-C4-S2.54, F.Cu at (413.2, 135.4)
- added H9: PZ254R-12-8P, easyeda_footprints:HDR-TH_8P-P2.54-H-M-R2-C4-S2.54, F.Cu at (424.6, 135.4)
- added J1: DB141V-2.54-4P, easyeda_footprints:CONN-TH_4P-P2.54_DIBO_DB141V-2.54-4P, F.Cu at (389.9, 140.6)
- added J2: DB141V-2.54-4P, easyeda_footprints:CONN-TH_4P-P2.54_DIBO_DB141V-2.54-4P, F.Cu at (389.9, 154.5)
- added J3: DB141V-2.54-4P, easyeda_footprints:CONN-TH_4P-P2.54_DIBO_DB141V-2.54-4P, F.Cu at (389.9, 168.4)
- added J4: DB141V-2.54-4P, easyeda_footprints:CONN-TH_4P-P2.54_DIBO_DB141V-2.54-4P, F.Cu at (287.7, 111.3)
- added Q12: YJQ10N2A, pauls_footprints:DFN2020-3, F.Cu at (422.3, 111.3)
- added Q3: YJQ10N2A, pauls_footprints:DFN2020-3, F.Cu at (422.3, 107.8)
- added Q4: YJQ10N2A, pauls_footprints:DFN2020-3, F.Cu at (409.4, 149.0)
- added Q5: YJQ10N2A, pauls_footprints:DFN2020-3, F.Cu at (409.4, 152.6)
- added Q6: YJQ10N2A, pauls_footprints:DFN2020-3, F.Cu at (409.4, 156.1)
- added Q7: YJQ10N2A, pauls_footprints:DFN2020-3, F.Cu at (409.4, 159.7)
- added Q8: JMTV210P02A, pauls_footprints:DFN2020-3, F.Cu at (400.5, 145.5)
- added R29: 10K, Resistor_SMD:R_0603_1608Metric, F.Cu at (400.5, 133.9)
- added R30: 10K, Resistor_SMD:R_0603_1608Metric, F.Cu at (400.5, 136.4)
- added R31: 1K, Resistor_SMD:R_0603_1608Metric, F.Cu at (400.5, 139.0)
- E1: footprint MB_Library:SMC_L6.9-W5.9-LS8.0-RD -> easyeda_footprints:SMC_L6.9-W5.9-LS8.0-RD
- LED1, LED10, LED11, LED12, LED13, LED14, LED15, LED16, LED17, LED18, LED19, LED2, LED20, LED21, LED22, LED23, LED24, LED25, LED26, LED27, LED28, LED29, LED3, LED30, LED31, LED32, LED33, LED34, LED35, LED36, LED37, LED38, LED39, LED4, LED40, LED41, LED42, LED43, LED44, LED45, LED46, LED47, LED48, LED5, LED6, LED7, LED8, LED9: value XL-2835UWC-02 -> XL-5730UWC-05; footprint MB_Library:LED-SMD_L3.5-W2.8-RD_1.25T-2PWT -> easyeda_footprints:LED-SMD_3P-L5.7-W3.0-RD
- Q1: value BC817 -> JMTV210P02A; footprint Package_TO_SOT_SMD:SOT-23 -> pauls_footprints:DFN2020-3; moved to F.Cu
- Q2: value SUD50P06-15-GE3 -> BC817; footprint MB_Library:TO-252-3_L6.5-W5.8-P4.58-BL -> Package_TO_SOT_SMD:SOT-23; moved to F.Cu
- R10, R12, R13, R14, R15, R16, R18, R20, R22, R23, R24, R25, R26, R7, R8: value FRC0805F30R0TS -> 18R; footprint MB_Library:R0805 -> Resistor_SMD:R_1210_3225Metric
- R17: value 30R -> 18R; footprint MB_Library:R0805 -> Resistor_SMD:R_1210_3225Metric
- R2, R3: footprint Capacitor_SMD:C_0805_2012Metric_Pad1.18x1.45mm_HandSolder -> Resistor_SMD:R_0805_2012Metric
- R4: value 0.1R/1% (PT2512FK-070R1L) -> 0.1R/1%; footprint MB_Library:R2512 -> Resistor_SMD:R_2512_6332Metric
- R5, R6: footprint MB_Library:R0603 -> Resistor_SMD:R_0603_1608Metric
- TP4: value +12VLED L -> LED L GND
- TP6: value +12VLED R -> LED R GND
- U10, U11, U13, U14: footprint MB_Library:SW-SMD_SMXS-08K-TP -> easyeda_footprints:SW-SMD_SMXS-08K-TP
- U2: footprint MB_Library:TO-263-5_L10.2-W8.9-P1.70-TL -> easyeda_footprints:TO-263-5_L10.2-W8.9-P1.70-TL
- U3: footprint MB_Library:SOT-23-8_L3.0-W1.7-P0.65-LS2.8-BR -> Package_TO_SOT_SMD:SOT-23-8
- U7: footprint MB_Library:HDR-TH_40P-P2.54-H-F-R2-C20-W8.5 -> easyeda_footprints:HDR-TH_40P-P2.54-H-F-R2-C20-W8.5
- moved R14 391.8 mm to (428.7, 95.5), turned to 0 degrees
- moved R16 390.2 mm to (428.7, 103.9)
- moved R7 380.5 mm to (423.1, 91.3), turned to 0 degrees
- moved R15 369.7 mm to (428.7, 99.7), turned to 0 degrees
- moved LED24 364.3 mm to (402.4, 103.7), turned to 0 degrees
- moved LED22 364.0 mm to (402.4, 95.4), turned to 0 degrees
- moved LED23 363.5 mm to (402.4, 99.6)
- moved LED18 358.9 mm to (395.3, 120.3)
- moved LED17 358.1 mm to (395.3, 116.2), turned to 0 degrees
- moved LED16 356.9 mm to (395.3, 112.0)
- moved R26 356.7 mm to (440.0, 103.9), turned to 0 degrees
- moved LED47 351.9 mm to (416.7, 116.2), turned to 0 degrees
- moved LED1 344.0 mm to (388.1, 91.3), turned to 0 degrees
- moved LED21 342.0 mm to (402.4, 91.3)
- moved LED19 335.3 mm to (395.3, 124.5)
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Connections:
- LED2 pad 1: Net-(LED2-K) -> Net-(LED1-A)
- LED2 pad 2: Net-(LED1-K) -> Net-(LED2-A)
- LED3 pad 2: Net-(LED2-K) -> Net-(LED1-K)
- LED48 pad 1: Net-(LED27-K) -> unconnected-(LED48-K-Pad1)
- Q1 pad 1: EN_12VReg -> Net-(Q1-G)
- Q1 pad 2: GND -> +24V
- Q1 pad 3: Net-(Q1-C) -> Net-(J3-Pin_3)
- Q2 pad 1: Net-(Q1-C) -> Net-(Q2-B)
- Q2 pad 2: Net-(Q2-D) -> GND
- Q2 pad 3: /Power/VIN- -> Net-(Q1-G)
- R10 pad 1: Net-(LED7-A) -> +12V
- R10 pad 2: +12V -> Net-(LED34-A)
- R12 pad 1: Net-(LED10-A) -> +12V
- R12 pad 2: +12V -> Net-(LED37-A)
- R13 pad 1: Net-(LED13-A) -> +12V
- R13 pad 2: +12V -> Net-(LED40-A)
- R14 pad 1: Net-(LED16-A) -> +12V
- R14 pad 2: +12V -> Net-(LED43-A)
- R15 pad 1: Net-(LED19-A) -> +12V
- R15 pad 2: +12V -> Net-(LED46-A)
- R16 pad 1: Net-(LED22-A) -> +12V
- R16 pad 2: +12V -> Net-(LED25-A)
- R17 pad 1: Net-(LED25-A) -> +12V
- R17 pad 2: +12V -> Net-(LED2-A)
- R18 pad 1: Net-(LED28-A) -> +12V
- R18 pad 2: +12V -> Net-(LED4-A)
- R20 pad 1: Net-(LED31-A) -> +12V
- R20 pad 2: +12V -> Net-(LED7-A)
- R22 pad 1: Net-(LED34-A) -> +12V
- R22 pad 2: +12V -> Net-(LED10-A)
- R23 pad 1: Net-(LED37-A) -> +12V
- R23 pad 2: +12V -> Net-(LED13-A)
- R24 pad 1: Net-(LED40-A) -> +12V
- R24 pad 2: +12V -> Net-(LED16-A)
- R25 pad 1: Net-(LED43-A) -> +12V
- R25 pad 2: +12V -> Net-(LED19-A)
- R26 pad 1: Net-(LED46-A) -> +12V
- R26 pad 2: +12V -> Net-(LED22-A)
- R4 pad 1: /Power/VIN+ -> +24V
- R4 pad 2: /Power/VIN- -> Net-(U3-IN+)
- R7 pad 1: Net-(LED1-A) -> +12V
- R7 pad 2: +12V -> Net-(LED28-A)
- R8 pad 1: Net-(LED4-A) -> +12V
- R8 pad 2: +12V -> Net-(LED31-A)
- U3 pad 1: /Power/VIN+ -> Net-(U3-IN+)
- U3 pad 2: /Power/VIN- -> +24V
Routing:
- net Net-(LED12-K): track 0.00 -> 393.8 mm
- net /Photo LED's/+12V_L_LED: track 393.8 -> 0.00 mm
- net Net-(LED27-K): track 0.00 -> 378.3 mm
- net /Photo LED's/+12V_R_LED: track 378.3 -> 0.00 mm
- net (no net): track 126.3 -> 218.2 mm, vias 1 -> 3
- net /Power/VIN-: track 37.0 -> 0.00 mm
- net Net-(Q2-D): track 28.3 -> 0.00 mm
- net GND: track 51.9 -> 38.4 mm
- net +3.3V: track 342.5 -> 356.1 mm
- net Net-(LED2-K): track 13.5 -> 0.00 mm
- net Net-(Q1-C): track 7.15 -> 0.00 mm, vias 2 -> 0
- net /Power/VIN+: track 5.93 -> 0.00 mm

Commit message: daily PCB update
Parts:
- B1: value ~ -> graphic; footprint AQLibrary:Talentcell -> MothBox_footprints_Library:Talentcell
- C1: footprint Capacitor_SMD:CP_Elec_10x12.5 -> MothBox_footprints_Library:CP_Elec_10x12.5
- C2, C3, C5: footprint Capacitor_SMD:C_0805_2012Metric_Pad1.18x1.45mm_HandSolder -> MothBox_footprints_Library:R_0603_1608Metric
- C4: footprint Capacitor_SMD:CP_Elec_10x10 -> MothBox_footprints_Library:CP_Elec_10x10
- C6: footprint Capacitor_SMD:C_0603_1608Metric -> MothBox_footprints_Library:C_0603_1608Metric; moved to B.Cu
- C7: footprint Capacitor_SMD:C_0805_2012Metric -> MothBox_footprints_Library:C_0603_1608Metric
- C9: footprint Capacitor_SMD:C_0805_2012Metric -> MothBox_footprints_Library:C_0603_1608Metric; moved to B.Cu
- D1, D2, D5, D6, D7: footprint Diode_SMD:D_SOD-323 -> MothBox_footprints_Library:D_SOD-323
- E1: footprint easyeda_footprints:SMC_L6.9-W5.9-LS8.0-RD -> MothBox_footprints_Library:SMC_L6.9-W5.9-LS8.0-RD
- F2: footprint Resistor_SMD:R_1812_4532Metric -> Fuse:Fuse_1812_4532Metric
- H1: value GPS 4 pin 2.54-1*4P母 -> GPS 4 pin 2.54-1*4P; footprint AQLibrary:GPS4pin_HDR-TH_4P-P2.54-V-F -> Connector_PinSocket_2.54mm:PinSocket_1x04_P2.54mm_Vertical
- H10, H8, H9: footprint easyeda_footprints:HDR-TH_8P-P2.54-H-M-R2-C4-S2.54 -> MothBox_footprints_Library:HDR-TH_8P-P2.54-H-M-R2-C4-S2.54
- H2, H3, H4, H5, H6, H7: footprint MountingHole:MountingHole_6.4mm_M6_Pad -> MothBox_footprints_Library:MountingHole_6.4mm_M6_Pad
- J1, J2, J3, J4: footprint easyeda_footprints:CONN-TH_4P-P2.54_DIBO_DB141V-2.54-4P -> MothBox_footprints_Library:CONN-TH_4P-P2.54_DIBO_DB141V-2.54-4P
- L1: footprint Inductor_SMD:L_Chilisin_BMRG00131360 -> MothBox_footprints_Library:L_Chilisin_BMRG00131360
- LED1, LED10, LED11, LED12, LED13, LED14, LED15, LED16, LED17, LED18, LED19, LED2, LED20, LED21, LED22, LED23, LED24, LED25, LED26, LED27, LED28, LED29, LED3, LED30, LED31, LED32, LED33, LED34, LED35, LED36, LED37, LED38, LED39, LED4, LED40, LED41, LED42, LED43, LED44, LED45, LED46, LED47, LED48, LED5, LED6, LED7, LED8, LED9: footprint easyeda_footprints:LED-SMD_3P-L5.7-W3.0-RD -> MothBox_footprints_Library:LED-SMD_3P-L5.7-W3.0-RD
- Q1, Q12, Q3, Q4, Q5, Q6, Q7, Q8: footprint pauls_footprints:DFN2020-3 -> MothBox_footprints_Library:DFN2020-3
- Q2: footprint Package_TO_SOT_SMD:SOT-23 -> MothBox_footprints_Library:SOT-23
- R10, R12, R13, R14, R15, R16, R17, R18, R20, R22, R23, R24, R25, R26, R7, R8: footprint Resistor_SMD:R_1210_3225Metric -> MothBox_footprints_Library:R_1210_3225Metric
- R11, R19, R2, R21, R27, R28, R3, R9: footprint Resistor_SMD:R_0805_2012Metric -> MothBox_footprints_Library:R_0805_2012Metric
- R29, R30, R31, R5, R6: footprint Resistor_SMD:R_0603_1608Metric -> MothBox_footprints_Library:R_0603_1608Metric
- R4: footprint Resistor_SMD:R_2512_6332Metric -> MothBox_footprints_Library:R_2512_6332Metric
- TP1, TP3, TP4, TP6: footprint TestPoint:TestPoint_THTPad_D1.0mm_Drill0.5mm -> MothBox_footprints_Library:TestPoint_THTPad_D1.0mm_Drill0.5mm
- U10, U11, U13, U14: footprint easyeda_footprints:SW-SMD_SMXS-08K-TP -> MothBox_footprints_Library:SW-SMD_SMXS-08K-TP
- U15, U16: footprint Package_SO:TSSOP-24_4.4x7.8mm_P0.65mm -> MothBox_footprints_Library:TSSOP-24_4.4x7.8mm_P0.65mm; moved to B.Cu
- U19: value ~ -> graphic; footprint Attractor:Arducam Owlsight -> MothBox_footprints_Library:Arducam Owlsight
- U2: footprint easyeda_footprints:TO-263-5_L10.2-W8.9-P1.70-TL -> MothBox_footprints_Library:TO-263-5_L10.2-W8.9-P1.70-TL
- U3: footprint Package_TO_SOT_SMD:SOT-23-8 -> MothBox_footprints_Library:SOT-23-8
- U5: footprint AQLibrary:EPAPER_PinHeader_2x20_P2.54mm_Vertical -> MothBox_footprints_Library:EPAPER_PinHeader_2x20_P2.54mm_Vertical
- U7: footprint easyeda_footprints:HDR-TH_40P-P2.54-H-F-R2-C20-W8.5 -> MothBox_footprints_Library:HDR-TH_40P-P2.54-H-F-R2-C20-W8.5
- U8: footprint AQLibrary:GPS5pin_HDR-TH_5P-P2.54-V-F -> Connector_PinSocket_2.54mm:PinSocket_1x05_P2.54mm_Vertical
- moved R26 394.0 mm to (46.2, 116.7), turned to 180 degrees
- moved R24 391.7 mm to (55.6, 170.7), turned to 180 degrees
- moved R25 372.1 mm to (68.7, 125.5), turned to -90 degrees
- moved R17 365.6 mm to (78.0, 173.2), turned to -90 degrees
- moved LED23 364.9 mm to (37.6, 103.6), turned to -90 degrees
- moved LED22 363.7 mm to (39.3, 114.8)
- moved LED24 362.8 mm to (39.8, 92.5), turned to 180 degrees
- moved LED16 356.5 mm to (44.3, 174.5)
- moved LED18 356.4 mm to (40.1, 149.8)
- moved LED17 352.5 mm to (45.7, 162.0), turned to -90 degrees
- moved LED21 346.4 mm to (61.2, 151.2)
- moved LED3 343.7 mm to (58.2, 195.9)
- moved LED1 339.8 mm to (60.3, 180.9), turned to 90 degrees
- moved R15 339.3 mm to (93.3, 151.0), turned to -90 degrees
- moved LED46 338.7 mm to (80.8, 155.7), turned to 90 degrees
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Connections:
- H8 pad 1: +12V -> unconnected-(H8-Pad1)
- H8 pad 2: unconnected-(H8-Pad2) -> +12V
- H8 pad 3: +12V -> unconnected-(H8-Pad3)
- H8 pad 4: unconnected-(H8-Pad4) -> +12V
- H8 pad 5: Net-(H8-Pad5) -> unconnected-(H8-Pad5)
- H8 pad 6: unconnected-(H8-Pad6) -> Net-(H8-Pad6)
- H8 pad 7: Net-(H8-Pad5) -> unconnected-(H8-Pad7)
- H8 pad 8: unconnected-(H8-Pad8) -> Net-(H8-Pad6)
- H9 pad 1: +12V -> unconnected-(H9-Pad1)
- H9 pad 2: unconnected-(H9-Pad2) -> +12V
- H9 pad 3: +12V -> unconnected-(H9-Pad3)
- H9 pad 4: unconnected-(H9-Pad4) -> +12V
- H9 pad 5: Net-(H9-Pad5) -> unconnected-(H9-Pad5)
- H9 pad 6: unconnected-(H9-Pad6) -> Net-(H9-Pad6)
- H9 pad 7: Net-(H9-Pad5) -> unconnected-(H9-Pad7)
- H9 pad 8: unconnected-(H9-Pad8) -> Net-(H9-Pad6)
- LED48 pad 1: unconnected-(LED48-K-Pad1) -> Net-(LED27-K)
- Q6 pad 1: Net-(H8-Pad5) -> Net-(H8-Pad6)
- Q6 pad 2: Net-(H8-Pad5) -> Net-(H8-Pad6)
- Q6 pad 3: Net-(H8-Pad5) -> Net-(H8-Pad6)
- Q7 pad 1: Net-(H9-Pad5) -> Net-(H9-Pad6)
- Q7 pad 2: Net-(H9-Pad5) -> Net-(H9-Pad6)
- Q7 pad 3: Net-(H9-Pad5) -> Net-(H9-Pad6)
- U15 pad 10: /GPS and Switches/Mon -> /GPS and Switches/Sat
- U15 pad 11: /GPS and Switches/Armed/Disarmed -> /GPS and Switches/Sun
- U15 pad 13: /GPS and Switches/Test_Debug -> /GPS and Switches/C2
- U15 pad 14: /GPS and Switches/HI/LOW_PWR -> /GPS and Switches/C1
- U15 pad 15: /GPS and Switches/INT/EXT_Attractor -> /GPS and Switches/Attractor_3
- U15 pad 16: /GPS and Switches/Attractor_1 -> /GPS and Switches/Attractor_2
- U15 pad 17: /GPS and Switches/Attractor_2 -> /GPS and Switches/Attractor_1
- U15 pad 18: /GPS and Switches/Attractor_3 -> /GPS and Switches/INT/EXT_Attractor
- U15 pad 19: /GPS and Switches/C1 -> /GPS and Switches/HI/LOW_PWR
- U15 pad 20: /GPS and Switches/C2 -> /GPS and Switches/Test_Debug
- U15 pad 4: /GPS and Switches/Sun -> /GPS and Switches/Armed/Disarmed
- U15 pad 5: /GPS and Switches/Sat -> /GPS and Switches/Mon
- U15 pad 6: /GPS and Switches/Fri -> /GPS and Switches/Tue
- U15 pad 7: /GPS and Switches/Thur -> /GPS and Switches/Wed
- U15 pad 8: /GPS and Switches/Wed -> /GPS and Switches/Thur
- U15 pad 9: /GPS and Switches/Tue -> /GPS and Switches/Fri
Routing:
- net +12V: track 520.3 -> 815.8 mm, vias 3 -> 17
- net SDA: track 403.6 -> 575.2 mm, vias 5 -> 9
- net SCL: track 404.5 -> 576.0 mm, vias 7 -> 11
- net unconnected-(U7-Pad16): track 180.6 -> 31.9 mm
- net unconnected-(U7-Pad35): track 148.5 -> 0.00 mm, vias 3 -> 0
- net unconnected-(U7-Pad11): track 165.9 -> 18.9 mm, vias 4 -> 2
- net unconnected-(U7-Pad14): track 181.7 -> 62.1 mm, vias 8 -> 4
- net (no net): track 218.2 -> 118.5 mm, vias 3 -> 1
- net +3.3V: track 356.1 -> 268.4 mm, vias 2 -> 1
- net unconnected-(U7-Pad34): track 193.6 -> 110.6 mm, vias 6 -> 4
- net Net-(LED27-K): track 378.3 -> 456.7 mm, vias 2 -> 0
- net Net-(LED7-K): track 42.6 -> 11.0 mm
- net Net-(LED12-K): track 393.8 -> 424.6 mm
- net +24V: track 56.3 -> 29.0 mm, vias 1 -> 0
- net Net-(LED43-A): track 3.06 -> 30.0 mm
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Other:
- board text added: "MOTHBOX V5.0.1"
- board text removed: "ATTRACTOR 1"
- board text removed: "MOTHBOX V5.0.0"
