File: Hardware/PCB/Andy_PCB_5.0.1/MothBox/Photo_LEDs.kicad_sch (KiCad schematic)
At the start: 71 parts, among them Q12 YJQ10N2A, Q3 YJQ10N2A

Commit message: updated photo LEDs and the power page
Parts:
- removed LED1, LED10, LED11, LED12, LED13, LED14, LED15, LED16, LED17, LED18, LED19, LED2, LED20, LED21, LED22, LED23, LED24, LED25, LED26, LED27, LED28, LED29, LED3, LED30, LED31, LED32, LED33, LED34, LED35, LED36, LED37, LED38, LED39, LED4, LED40, LED41, LED42, LED43, LED44, LED45, LED46, LED47, LED48, LED5, LED6, LED7, LED8, LED9: XL-2835UWC-02, easyeda2kicad:LED-SMD_L3.5-W2.8-RD_1.25T-2PWT, symbol MB_Library:XL-2835UWC-02
- removed R10, R12, R13, R14, R15, R16, R18, R20, R22, R23, R24, R25, R26, R7, R8: FRC0805F30R0TS, easyeda2kicad:R0805, symbol MB_Library:FRC0805F30R0TS
- removed R17: 30R, easyeda2kicad:R0805, symbol MB_Library:FRC0805F30R0TS
- added LED1, LED10, LED11, LED12, LED13, LED14, LED15, LED16, LED17, LED18, LED19, LED2, LED20, LED21, LED22, LED23, LED24, LED25, LED26, LED27, LED28, LED29, LED3, LED30, LED31, LED32, LED33, LED34, LED35, LED36, LED37, LED38, LED39, LED4, LED40, LED41, LED42, LED43, LED44, LED45, LED46, LED47, LED48, LED5, LED6, LED7, LED8, LED9: XL-5730UWC-05, easyeda2kicad:LED-SMD_3P-L5.7-W3.0-RD, symbol easyeda_libraries:XL-5730UWC-05
- added R10, R12, R13, R14, R15, R16, R17, R18, R20, R22, R23, R24, R25, R26, R7, R8: 18R, Resistor_SMD:R_1210_3225Metric, symbol MB_Library:R_Small
- TP4: value +12VLED L -> LED L GND
- TP6: value +12VLED R -> LED R GND
Connections:
- net +12V: now also R10.1, R12.1, R13.1, R14.1, R15.1, R16.1, R17.1, R18.1, R20.1, R22.1, R23.1, R24.1, R25.1, R26.1, R7.1, R8.1
- net at Q3.1 (D), Q3.2 (D), Q3.3 (D)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: now also LED27.1 (K), LED30.1 (K), LED33.1 (K), LED36.1 (K), LED39.1 (K), LED42.1 (K), LED45.1 (K)
- net at Q12.1 (D), Q12.2 (D), Q12.3 (D)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: now also LED12.1 (K), LED15.1 (K), LED18.1 (K), LED21.1 (K), LED24.1 (K), LED3.1 (K), LED6.1 (K), LED9.1 (K)
- new net: LED17.1 (K), LED18.2 (A)
- new net: LED11.1 (K), LED12.2 (A)
- new net: LED10.1 (K), LED11.2 (A)
- new net: LED1.1 (K), LED3.2 (A)
- new net: LED1.2 (A), LED2.1 (K)
- new net: LED26.1 (K), LED27.2 (A)
- new net: LED7.1 (K), LED8.2 (A)
- new net: LED7.2 (A), R20.2
- new net: LED31.1 (K), LED32.2 (A)
- new net: LED31.2 (A), R8.2
- new net: LED5.1 (K), LED6.2 (A)
- new net: LED40.2 (A), R13.2
- new net: LED2.2 (A), R17.2
- new net: LED44.1 (K), LED45.2 (A)
- new net: LED43.1 (K), LED44.2 (A)
- new net: LED35.1 (K), LED36.2 (A)
- new net: LED34.1 (K), LED35.2 (A)
- new net: LED28.2 (A), R7.2
- new net: LED25.2 (A), R16.2
- new net: LED38.1 (K), LED39.2 (A)
- new net: LED37.1 (K), LED38.2 (A)
- new net: LED25.1 (K), LED26.2 (A)
- new net: LED20.1 (K), LED21.2 (A)
- new net: LED13.2 (A), R23.2
- new net: LED37.2 (A), R12.2
- new net: LED13.1 (K), LED14.2 (A)
- new net: LED47.1 (K), LED48.2 (A)
- new net: LED46.1 (K), LED47.2 (A)
- new net: LED16.2 (A), R24.2
- new net: LED40.1 (K), LED41.2 (A)
- new net: LED4.2 (A), R18.2
- new net: LED32.1 (K), LED33.2 (A)
- new net: LED10.2 (A), R22.2
- new net: LED41.1 (K), LED42.2 (A)
- new net: LED22.1 (K), LED23.2 (A)
- new net: LED22.2 (A), R26.2
- new net: LED16.1 (K), LED17.2 (A)
- new net: LED23.1 (K), LED24.2 (A)
- new net: LED4.1 (K), LED5.2 (A)
- new net: LED29.1 (K), LED30.2 (A)
- new net: LED19.1 (K), LED20.2 (A)
- new net: LED19.2 (A), R25.2
- new net: LED46.2 (A), R15.2
- new net: LED34.2 (A), R10.2
- new net: LED14.1 (K), LED15.2 (A)
- new net: LED8.1 (K), LED9.2 (A)
- new net: LED28.1 (K), LED29.2 (A)
- new net: LED43.2 (A), R14.2
- no-connect marks 0 -> 47
Other:
- note added: "v5.0.0 used XINGLIGHT XL-2835UWC-02 60mA 6000K~7500K Yellow lens -20℃~+85℃ Positive Stick White 120° 200mW 3.4V SMD2835 LED Indication - Discrete ROH Figure out: Each string used around 83mA how many batches per transistor thing what is the light angle of these LEDS (if any) without lens is cheaper Current per led = 60mA Total current = 8(columns) x 60mA = 480mA Total Luminous required = ?? lm Pe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"
- note added: "v5.0.1 used the XL-2835UWC-02 it should draw around 133mA at 12V therefore each bank should draw 1.072A, or 2.144A total"
- note removed: "30R"
- note removed: "PH: Measure the current flowing through the LED strings. Does the resistance need to be modified?"
- note removed: "XINGLIGHT XL-2835UWC-02 60mA 6000K~7500K Yellow lens -20℃~+85℃ Positive Stick White 120° 200mW 3.4V SMD2835 LED Indication - Discrete ROH Figure out: How much current do these LEDs need how many batches per transistor thing what is the light angle of these LEDS (if any) without lens is cheaper Current per led = 60mA Total current = 8(columns) x 60mA = 480mA Total Luminous required = ?? lm Per led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"
- company: (none) -> Digital Naturalism Laboritories
- title: (none) -> MothBox
- moved on the sheet: Q12, Q3, R11, R9, TP3, TP4, TP6

Commit message: updated footprints and schematic
Parts:
- LED1, LED10, LED11, LED12, LED13, LED14, LED15, LED16, LED17, LED18, LED19, LED2, LED20, LED21, LED22, LED23, LED24, LED25, LED26, LED27, LED28, LED29, LED3, LED30, LED31, LED32, LED33, LED34, LED35, LED36, LED37, LED38, LED39, LED4, LED40, LED41, LED42, LED43, LED44, LED45, LED46, LED47, LED48, LED5, LED6, LED7, LED8, LED9: footprint easyeda2kicad:LED-SMD_3P-L5.7-W3.0-RD -> easyeda_footprints:LED-SMD_3P-L5.7-W3.0-RD; symbol easyeda_libraries:XL-5730UWC-05 -> MothBox_Symbol_Library:XL-5730UWC-05; LCSC Part C2843887 -> (none); LCSC_Part (none) -> C2843887
- Q12: footprint Pauls_Footprints:DFN2020-3 -> pauls_footprints:DFN2020-3; symbol _pauls_library:YJQ10N2A -> MothBox_Symbol_Library:YJQ10N2A_1_1_1
- Q3: footprint Pauls_Footprints:DFN2020-3 -> pauls_footprints:DFN2020-3; symbol _pauls_library:YJQ10N2A -> MothBox_Symbol_Library:YJQ10N2A_2_1_1
- R10, R12, R13, R14, R15, R16, R17, R18, R20, R22, R23, R24, R25, R26, R7, R8: symbol MB_Library:R_Small -> MothBox_Symbol_Library:R_Small
- R11, R9: symbol MB_Library:R_US -> MothBox_Symbol_Library:R_US; LCSC Part no  C84376 -> (none); LCSC_Part_No (none) -> C84376
- TP3, TP4, TP6: symbol MB_Library:TestPoint -> MothBox_Symbol_Library:TestPoint

Commit message: daily PCB update
Parts:
- LED1, LED10, LED11, LED12, LED13, LED14, LED15, LED16, LED17, LED18, LED19, LED2, LED20, LED21, LED22, LED23, LED24, LED25, LED26, LED27, LED28, LED29, LED3, LED30, LED31, LED32, LED33, LED34, LED35, LED36, LED37, LED38, LED39, LED4, LED40, LED41, LED42, LED43, LED44, LED45, LED46, LED47, LED48, LED5, LED6, LED7, LED8, LED9: footprint easyeda_footprints:LED-SMD_3P-L5.7-W3.0-RD -> MothBox_footprints_Library:LED-SMD_3P-L5.7-W3.0-RD
- Q12: footprint pauls_footprints:DFN2020-3 -> MothBox_footprints_Library:DFN2020-3; symbol MothBox_Symbol_Library:YJQ10N2A_1_1_1 -> MothBox_Symbol_Library:YJQ10N2A_1_1_1_1_1
- Q3: footprint pauls_footprints:DFN2020-3 -> MothBox_footprints_Library:DFN2020-3; symbol MothBox_Symbol_Library:YJQ10N2A_2_1_1 -> MothBox_Symbol_Library:YJQ10N2A_2_1_1_1_1
- R10, R12, R13, R14, R15, R16, R17, R18, R20, R22, R23, R24, R25, R26, R7, R8: footprint Resistor_SMD:R_1210_3225Metric -> MothBox_footprints_Library:R_1210_3225Metric
- R11, R9: footprint Resistor_SMD:R_0805_2012Metric -> MothBox_footprints_Library:R_0805_2012Metric
- TP3, TP4, TP6: footprint TestPoint:TestPoint_THTPad_D1.0mm_Drill0.5mm -> MothBox_footprints_Library:TestPoint_THTPad_D1.0mm_Drill0.5mm
Connections:
- net at LED27.1 (K), LED30.1 (K), LED33.1 (K)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: now also LED48.1 (K)
Other:
- note added: "wrong symbol pins"
- moved on the sheet: LED28, LED29, LED30, LED31, LED32, LED33, LED34, LED35, LED36, LED37, LED38, LED39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

Commit message: rough outline of PCB. Lots of tidying up needed
Parts:
- removed Q12: YJQ10N2A, MothBox_footprints_Library:DFN2020-3, symbol MothBox_Symbol_Library:YJQ10N2A_1_1_1_1_1
- removed Q3: YJQ10N2A, MothBox_footprints_Library:DFN2020-3, symbol MothBox_Symbol_Library:YJQ10N2A_2_1_1_1_1
- removed R11, R9: 10k, MothBox_footprints_Library:R_0805_2012Metric, symbol MothBox_Symbol_Library:R_US
- added Q3, Q7: YJQ10N2A, MothBox_footprints_Library:U-DFN2020-6_L2.0-W2.0-P0.65-BL, symbol MothBox_Symbol_Library:YJQ10N2A_1
- added R11, R9: 10K, MothBox_footprints_Library:R_0603_1608Metric, symbol MothBox_Symbol_Library:R_Small
Connections:
- net GND: now also Q3.4 (S), Q3.7 (S), Q7.4 (S), Q7.7 (S), R11.2, R9.2
- net PHOTO_LED_CTRL: now also Q3.3 (G), Q7.3 (G), R11.1, R9.1
- net at LED12.1 (K), LED15.1 (K), LED18.1 (K)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: now also Q3.1 (D), Q3.2 (D), Q3.5 (D), Q3.6 (D), Q3.8 (D)
- net at LED27.1 (K), LED30.1 (K), LED33.1 (K)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: now also Q7.1 (D), Q7.2 (D), Q7.5 (D), Q7.6 (D), Q7.8 (D)
Other:
- note removed: "wrong symbol pins"

Commit message: added in extra hour switch for 24hr coverage
Parts:
- Q3, Q7: LCSC C919558 -> (none); LCSC_Part (none) -> C919558
- R10, R12, R13, R14, R15, R16, R17, R18, R20, R22, R23, R24, R25, R26, R7, R8: LCSC C48392080 -> (none); LCSC_Part (none) -> C48392080
- R11, R9: LCSC_Part (none) -> C25804
- TP3, TP4, TP6: now left out of the parts list
