File: Hardware/PCB/Andy_PCB_5.0.2/MothBox/RPI5.kicad_sch (KiCad schematic)
At the start: 5 parts, among them U4 RASPBERRY_PI_4B_4GB, U5 RASPBERRY_PI_5, U6 RASPBERRY_PI_4B_4GB, U7 Female Inv Socket Pi 2.54-2*20

Commit message: updating for v5.0.2
Parts:
- removed TP7: 3V3_test, MothBox_footprints_Library:TestPoint_THTPad_D1.0mm_Drill0.5mm, symbol MothBox_Symbol_Library:TestPoint
- added C1: 1000uF 50V, 0_easyeda_footprints:CAP-TH_BD16.0-P7.50-D1.2-FD, symbol MothBox_Symbol_Library:C_Polarized_Small_US
- added C17, C18: 10uF, MothBox_footprints_Library:C_0603_1608Metric, symbol MothBox_Symbol_Library:C_Small
Connections:
- net +5V: now also C1.1
- net GND: now also C1.2, C17.2, C18.2
- net 3V3_CTL: now reaches U7.14
- removed net +3.3V: U5.1 (3V3), U5.17 (3V3), U7.2
- net GPIO4/GPIO_GCKL: no longer names the net of U5.7 (GPIO4/GPIO_GCKL)
- net GPIO4/GPIO_GCKL: no longer U7.8
- new net +3V3: C17.1, C18.1, U7.2
- new net GPIO4: U7.8
- no-connect marks 24 -> 26

Commit message: final updates to v5.0.2 after error checking
Connections:
- net User_LED: now reaches U7.34
- net SWITCH: now reaches U7.35
- no-connect marks 26 -> 24
Other:
- note added: "1"
- note added: "11"
- note added: "12"
- note added: "13"
- note added: "15"
- note added: "2"
- note added: "3.3V"
- note added: "7"
- note added: "8"
- note added: "NOTE: The connector is in back-to-front. But it's wired up so it works."
Changed lines of the file:
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@@
 	(title_block
 		(title "MothBox")
-		(date "2025-09-29")
+		(date "2025-10-02")
 		(rev "5.0.2")
 		(company "Digital Naturalism Laboritories")
@@
 		)
 	)
+	(text "13"
+		(exclude_from_sim no)
+		(at 241.554 68.58 0)
+		(effects
+			(font
+				(size 1.27 1.27)
+				(thickness 0.254)
+				(bold yes)
+			)
+		)
+	)
+	(text "2"
+		(exclude_from_sim no)
+		(at 260.858 53.086 0)
+		(effects
+			(font
+				(size 1.27 1.27)
+				(thickness 0.254)
+				(bold yes)
+			)
+		)
+	)
+	(text "1"
+		(exclude_from_sim no)
+		(at 241.808 53.086 0)
+		(effects
+			(font
+				(size 1.27 1.27)
+				(thickness 0.254)
+				(bold yes)
+			)
+		)
+	)
 	(text "Raspberry Pi 5\nConnector"
 		(exclude_from_sim no)
@@
 		)
 	)
+	(text "NOTE: The connector is in back-to-front.  \nBut it's wired up so it works."
+		(exclude_from_sim no)
+		(at 252.73 117.602 0)
+		(effects
+			(font
+				(size 2 2)
+				(thickness 0.4)
+				(bold yes)
+				(color 255 19 27 1)
+			)
+		)
+	)
 	(text "RPI 5 Module\n"
 		(exclude_from_sim no)
@@
 		)
 	)
+	(text "11"
+		(exclude_from_sim no)
+		(at 241.046 66.04 0)
+		(effects
+			(font
+				(size 1.27 1.27)
+				(thickness 0.254)
+				(bold yes)
+			)
+		)
+	)
+	(text "8"
+		(exclude_from_sim no)
+		(at 260.858 61.214 0)
+		(effects
+			(font
+				(size 1.27 1.27)
+				(thickness 0.254)
+				(bold yes)
+			)
+		)
+	)
+	(text "3.3V"
+		(exclude_from_sim no)
+		(at 237.744 75.184 0)
+		(effects
+			(font
+				(size 1.27 1.27)
+				(thickness 0.254)
+				(bold yes)
+			)
+		)
+	)
+	(text "15"
+		(exclude_from_sim no)
+		(at 241.808 71.374 0)
+		(effects
+			(font
+				(size 1.27 1.27)
+				(thickness 0.254)
+				(bold yes)
+			)
+		)
+	)
+	(text "12"
+		(exclude_from_sim no)
+		(at 261.112 66.04 0)
+		(effects
+			(font
+				(size 1.27 1.27)
+				(thickness 0.254)
+				(bold yes)
+			)
+		)
+	)
 	(text "Raspberry Pi 5\nePaper Hat"
 		(exclude_from_sim no)
@@
 		)
 	)
+	(text "2"
+		(exclude_from_sim no)
+		(at 241.808 56.134 0)
+		(effects
+			(font
+				(size 1.27 1.27)
+				(thickness 0.254)
+				(bold yes)
+			)
+		)
+	)
+	(text "7"
+		(exclude_from_sim no)
+		(at 242.316 61.468 0)
+		(effects
+			(font
+				(size 1.27 1.27)
+				(thickness 0.254)
+				(bold yes)
+			)
+		)
+	)
 	(junction
 		(at 135.89 123.19)
@@
 	)
 	(no_connect
+		(at 241.3 74.93)
+	)
+	(no_connect
+		(at 83.82 109.22)
+	)
+	(no_connect
+		(at 134.62 68.58)
+	)
+	(no_connect
+		(at 134.62 60.96)
+	)
+	(no_connect
+		(at 83.82 93.98)
+	)
+	(no_connect
+		(at 241.3 72.39)
+	)
+	(no_connect
+		(at 134.62 76.2)
+	)
+	(no_connect
+		(at 83.82 76.2)
+	)
+	(no_connect
+		(at 134.62 81.28)
+	)
+	(no_connect
+		(at 83.82 66.04)
+	)
+	(no_connect
+		(at 83.82 101.6)
+	)
+	(no_connect
+		(at 134.62 78.74)
+	)
+	(no_connect
+		(at 83.82 73.66)
+	)
+	(no_connect
+		(at 83.82 106.68)
+	)
+	(no_connect
+		(at 261.62 87.63)
+	)
+	(no_connect
+		(at 134.62 86.36)
+	)
+	(no_connect
+		(at 83.82 78.74)
+	)
+	(no_connect
+		(at 134.62 66.04)
+	)
+	(no_connect
+		(at 134.62 73.66)
+	)
+	(no_connect
+		(at 241.3 87.63)
+	)
+	(no_connect
+		(at 134.62 63.5)
+	)
+	(no_connect
+		(at 134.62 83.82)
+	)
+	(no_connect
 		(at 261.62 67.31)
-	)
-	(no_connect
-		(at 241.3 72.39)
-	)
-	(no_connect
-		(at 83.82 109.22)
-	)
-	(no_connect
-		(at 134.62 68.58)
-	)
-	(no_connect
-		(at 134.62 60.96)
-	)
-	(no_connect
-		(at 83.82 93.98)
-	)
-	(no_connect
-		(at 134.62 76.2)
-	)
-	(no_connect
-		(at 83.82 76.2)
-	)
-	(no_connect
-		(at 134.62 81.28)
-	)
-	(no_connect
-		(at 83.82 66.04)
-	)
-	(no_connect
-		(at 83.82 101.6)
-	)
-	(no_connect
-		(at 241.3 74.93)
-	)
-	(no_connect
-		(at 261.62 97.79)
-	)
-	(no_connect
-		(at 134.62 78.74)
-	)
-	(no_connect
-		(at 83.82 73.66)
-	)
-	(no_connect
-		(at 83.82 106.68)
-	)
-	(no_connect
-		(at 261.62 87.63)
-	)
-	(no_connect
-		(at 134.62 86.36)
-	)
-	(no_connect
-		(at 83.82 78.74)
-	)
-	(no_connect
-		(at 134.62 66.04)
-	)
-	(no_connect
-		(at 134.62 73.66)
-	)
-	(no_connect
-		(at 241.3 95.25)
-	)
-	(no_connect
-		(at 241.3 87.63)
-	)
-	(no_connect
-		(at 134.62 63.5)
-	)
-	(no_connect
-		(at 134.62 83.82)
 	)
 	(wire
@@
 				(hide yes)
 			)
+		)
+	)
+	(global_label "User_LED"
+		(shape input)
+		(at 241.3 95.25 180)
+		(fields_autoplaced yes)
+		(effects
+			(font
+				(size 1.27 1.27)
+			)
+			(justify right)
+		)
+		(property "Intersheetrefs" "${INTERSHEET_REFS}"
+			(at 229.6667 95.25 0)
+			(effects
+				(font
+					(size 1.27 1.27)
+				)
+				(justify right)
+				(hide yes)
+			)
+		)
+	)
+	(global_label "SWITCH"
+		(shape input)
+		(at 261.62 97.79 0)
+		(fields_autoplaced yes)
+		(effects
+			(font
+				(size 1.27 1.27)
+			)
+			(justify left)
+		)
+		(property "Intersheetrefs" "${INTERSHEET_REFS}"
+			(at 271.439 97.79 0)
+			(effects
+				(font
+					(size 1.27 1.27)
+				)
+				(justify left)
+				(hide yes)
+			)
