File: Hardware/PCB/Andy_PCB_5.0.2/MothBox/UV_LED_PCB.kicad_sch (KiCad schematic)
At the start: 19 parts, among them J4 DB141V-2.54-4P, Q4 YJQ10N2A, Q5 YJQ10N2A, Q6 YJQ10N2A, Q9 YJQ10N2A

Commit message: final updates to v5.0.2 after error checking
Changed lines of the file:
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@@
 	(title_block
 		(title "MothBox")
-		(date "2025-09-29")
+		(date "2025-10-02")
 		(rev "5.0.2")
 		(company "Digital Naturalism Laboritories")
@@
 		)
 	)
+	(text "-"
+		(exclude_from_sim no)
+		(at 108.966 121.158 0)
+		(effects
+			(font
+				(size 2 2)
+				(thickness 0.4)
+				(bold yes)
+			)
+		)
+	)
 	(text "UV External Attractor"
 		(exclude_from_sim no)
@@
 			(font
 				(size 1.27 1.27)
+			)
+		)
+	)
+	(text "-"
+		(exclude_from_sim no)
+		(at 107.696 56.388 0)
+		(effects
+			(font
+				(size 2 2)
+				(thickness 0.4)
+				(bold yes)
+			)
+		)
+	)
+	(text "+"
+		(exclude_from_sim no)
+		(at 233.172 49.53 0)
+		(effects
+			(font
+				(size 2 2)
+				(thickness 0.4)
+				(bold yes)
+			)
+		)
+	)
+	(text "+"
+		(exclude_from_sim no)
+		(at 107.696 51.054 0)
+		(effects
+			(font
+				(size 2 2)
+				(thickness 0.4)
+				(bold yes)
 			)
 		)
@@
 		)
 	)
+	(text "-"
+		(exclude_from_sim no)
+		(at 233.172 54.864 0)
+		(effects
+			(font
+				(size 2 2)
+				(thickness 0.4)
+				(bold yes)
+			)
+		)
+	)
 	(text "UV PCB2 current consumtiom = 500mA"
 		(exclude_from_sim no)
@@
 		(effects
 			(font
+				(size 2 2)
+				(thickness 0.4)
+				(bold yes)
+			)
+		)
+	)
+	(text "+"
+		(exclude_from_sim no)
+		(at 108.966 115.824 0)
+		(effects
+			(font
