File: Hardware/PCB/Andy_PCB_5.0.2/MothBox/Power.kicad_sch (KiCad schematic)
At the start: 36 parts, among them J1 DB141V-2.54-4P, J2 DB141V-2.54-4P, J3 DB141V-2.54-4P, Q1 JMTV210P02A, Q2 AO3400A, Q8 JMTV210P02A, U1 Place Holder voltage regulator, U2 XL4015E1, U3 INA219BIDCNT

Commit message: partial update on v5.0.2 modifications
Parts:
- R3: value 3.3K -> 3.0K; LCSC_Part C22978 -> C4211
Connections:
- net +12V: now also J1.3 (Pin_3), J1.4 (Pin_4); no longer J1.1 (Pin_1), J1.2 (Pin_2)
- net GND: now also J1.1 (Pin_1), J1.2 (Pin_2); no longer J1.3 (Pin_3), J1.4 (Pin_4)
Other:
- note added: "Buck Convertor (Input <9V-36V> PWR to +5.2V)"
- note added: "Up to 4A output at 5.2V"
- note removed: "Buck Convertor (Input <9V-36V> PWR to +5V)"
- note removed: "Up to 4A output at 5V"
Changed lines of the file:
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@@
 		)
 	)
-	(text "Buck Convertor (Input <9V-36V> PWR to +5V)"
+	(text "Buck Convertor (Input <9V-36V> PWR to +5.2V)"
 		(exclude_from_sim no)
 		(at 71.12 121.158 0)
@@
 		)
 	)
-	(text "Up to 4A output at 5V"
+	(text "Up to 4A output at 5.2V"
 		(exclude_from_sim no)
 		(at 135.382 126.492 0)
@@
 	)
 	(junction
-		(at 214.63 78.74)
-		(diameter 0)
-		(color 0 0 0 0)
-	)
-	(junction
 		(at 100.33 54.61)
 		(diameter 0)
@@
 	)
 	(junction
-		(at 214.63 81.28)
-		(diameter 0)
-		(color 0 0 0 0)
-	)
-	(junction
 		(at 154.94 138.43)
 		(diameter 0)
@@
 	)
 	(junction
+		(at 214.63 78.74)
+		(diameter 0)
+		(color 0 0 0 0)
+	)
+	(junction
 		(at 130.81 46.99)
 		(diameter 0)
@@
 	)
 	(junction
+		(at 214.63 81.28)
+		(diameter 0)
+		(color 0 0 0 0)
+	)
+	(junction
 		(at 210.82 77.47)
 		(diameter 0)
@@
 	)
 	(junction
-		(at 134.62 152.4)
+		(at 214.63 83.82)
 		(diameter 0)
 		(color 0 0 0 0)
 	)
 	(junction
-		(at 137.16 138.43)
+		(at 134.62 152.4)
 		(diameter 0)
 		(color 0 0 0 0)
 	)
 	(junction
-		(at 130.81 74.93)
+		(at 137.16 138.43)
 		(diameter 0)
 		(color 0 0 0 0)
 	)
 	(junction
-		(at 214.63 83.82)
+		(at 130.81 74.93)
 		(diameter 0)
 		(color 0 0 0 0)
@@
 	(wire
 		(pts
+			(xy 214.63 78.74) (xy 214.63 81.28)
+		)
+		(stroke
+			(width 0)
+			(type default)
+		)
+	)
+	(wire
+		(pts
 			(xy 147.32 143.51) (xy 147.32 138.43)
 		)
@@
 	(wire
 		(pts
-			(xy 214.63 77.47) (xy 214.63 78.74)
-		)
-		(stroke
-			(width 0)
-			(type default)
-		)
-	)
-	(wire
-		(pts
 			(xy 137.16 45.72) (xy 137.16 46.99)
 		)
@@
 	(wire
 		(pts
-			(xy 214.63 78.74) (xy 214.63 81.28)
+			(xy 214.63 77.47) (xy 214.63 78.74)
 		)
 		(stroke
@@
 			)
 		)
-		(property "Value" "3.3K"
+		(property "Value" "3.0K"
 			(at 123.19 152.3999 0)
 			(effects
@@
 			)
 		)
-		(property "LCSC_Part" "C22978"
+		(property "LCSC_Part" "C4211"
 			(at 120.65 151.13 0)
 			(effects
@@
 	(symbol
 		(lib_id "MothBox_Symbol_Library:Conn_01x04")
-		(at 219.71 81.28 0)
+		(at 219.71 83.82 0)
+		(mirror x)
 		(unit 1)
 		(exclude_from_sim no)
@@
 		(dnp no)
 		(property "Reference" "J1"
-			(at 218.186 76.2 0)
+			(at 218.186 88.9 0)
 			(effects
 				(font
@@
 		)
 		(property "Value" "DB141V-2.54-4P"
-			(at 212.598 89.408 0)
+			(at 215.9 91.44 0)
 			(effects
 				(font
@@
 		)
 		(property "Footprint" "MothBox_footprints_Library:CONN-TH_4P-P2.54_DIBO_DB141V-2.54-4P"
-			(at 219.71 81.28 0)
+			(at 219.71 83.82 0)
 			(effects
 				(font
@@
 		)
 		(property "Datasheet" "~"
-			(at 219.71 81.28 0)
+			(at 219.71 83.82 0)
 			(effects
 				(font
@@
 		)
 		(property "Description" "Generic connector, single row, 01x04, script generated (kicad-library-utils/schlib/autogen/connector/)"
-			(at 219.71 81.28 0)
+			(at 219.71 83.82 0)
 			(effects
 				(font
@@
 		)
 		(property "LCSC" ""
-			(at 219.71 81.28 0)
+			(at 219.71 83.82 0)
 			(effects
 				(font
@@
 		)
 		(property "AVAILABILITY" ""
-			(at 219.71 81.28 0)
+			(at 219.71 83.82 0)
 			(effects
 				(font
@@
 		)
 		(property "DESCRIPTION" ""
-			(at 219.71 81.28 0)
+			(at 219.71 83.82 0)
 			(effects
 				(font
@@
 		)
 		(property "Link" ""
-			(at 219.71 81.28 0)
+			(at 219.71 83.82 0)
 			(effects
 				(font
@@
 		)
 		(property "PACKAGE" ""
-			(at 219.71 81.28 0)
+			(at 219.71 83.82 0)
 			(effects
 				(font
@@
 		)
 		(property "PRICE" ""
-			(at 219.71 81.28 0)
+			(at 219.71 83.82 0)
 			(effects
 				(font
@@
 		)
 		(property "Ali_Express_Link" ""
-			(at 219.71 81.28 0)
+			(at 219.71 83.82 0)
 			(effects
 				(font
@@
 		)
 		(property "LCSC_PN" ""
-			(at 219.71 81.28 0)
+			(at 219.71 83.82 0)
 			(effects
 				(font
@@
 		)
 		(property "LCSC_Part" "C2898746"
-			(at 219.71 81.28 0)
+			(at 219.71 83.82 0)
 			(effects
 				(font
@@
 		)
 		(property "Sim.Device" ""
-			(at 219.71 81.28 0)
+			(at 219.71 83.82 0)
 			(effects
 				(font
@@
 		)
 		(property "Sim.Pins" ""
-			(at 219.71 81.28 0)
+			(at 219.71 83.82 0)
 			(effects
 				(font
@@
 		)
 		(property "Sim.Type" ""
-			(at 219.71 81.28 0)
+			(at 219.71 83.82 0)
 			(effects
 				(font

Commit message: updating for v5.0.2
Parts:
- removed C1, C4: 470uF 50V, MothBox_footprints_Library:CP_Elec_10x12.5, symbol MothBox_Symbol_Library:C_Polarized_Small_US
- added C14, C16: 1000uF 50V, 0_easyeda_footprints:CAP-TH_BD16.0-P7.50-D1.2-FD, symbol MothBox_Symbol_Library:C_Polarized_Small_US
- added C15: 0.1uF, MothBox_footprints_Library:C_0603_1608Metric, symbol MothBox_Symbol_Library:C_Small
- added D3: Green, symbol 0_pauls_symbols:Device_LED_Small
- added R32: 0R, MothBox_footprints_Library:R_0603_1608Metric, symbol MothBox_Symbol_Library:R_Small
- added R34: 3.0K, MothBox_footprints_Library:R_0603_1608Metric, symbol MothBox_Symbol_Library:R_Small
- added R35: 10K, MothBox_footprints_Library:R_0603_1608Metric, symbol MothBox_Symbol_Library:R_Small
Connections:
- net +24V: now also C14.1
- net +3.3V: now also R35.1
- net +5V: now also C16.1
- net GND: now also C14.2, C15.2, C16.2, D3.1 (K), R32.2; no longer R3.2
- new net: D3.2 (A), R34.2
- new net: C15.1, R35.2
- new net: R3.2, R32.1
Other:
- note added: "USER LED/Switch"
- note added: "Use for fine adjustments"

Commit message: final updates to v5.0.2 after error checking
Parts:
- added SW2: KH-6X6X5H-STM, 0_easyeda_footprints:SW-SMD_4P-L6.0-W6.0-P4.50-LS9.0_H5.0, symbol 0_easyeda2kicad:KH-6X6X5H-STM
- D3: footprint (none) -> LED_SMD:LED_0603_1608Metric; LCSC (none) -> C72043
Connections:
- net GND: now also SW2.3, SW2.4
- net SWITCH: now reaches C15.1, R35.2
- net SWITCH: now also SW2.1, SW2.2
- net User_LED: now reaches R34.1
Other:
- moved on the sheet: C15

Commit message: andy tweaked and passes DRC
Connections:
- net +3.3V: no longer R35.1
- new net +3V3: R35.1
Changed lines of the file:
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@@
 			)
 		)
-		(property "Value" "+3.3V"
+		(property "Value" "+3V3"
 			(at 260.858 111.76 0)
 			(effects
