File: Hardware/PCB/Andy_PCB_5.0.3/MothBox/MothBox_5.0.3/Power.kicad_sch (KiCad schematic)
At the start: 44 parts, among them J1 DB141V-2.54-4P, J2 DB141V-2.54-4P, J3 DB141V-2.54-4P, Q1 JMTV210P02A, Q2 AO3400A, Q8 JMTV210P02A, SW2 KH-6X6X5H-STM, U1 Place Holder voltage regulator, U2 XL4015E1, U3 INA219BIDCNT

Commit message: version 5.0.3 completed changes, as per CHANGELOG
Parts:
- added D2, D4: 6.8V, MothBox_footprints_Library:D_SOD-323, symbol MothBox_Symbol_Library:D_Zener_Small
- added Q10: JMTV210P02A, MothBox_footprints_Library:U-DFN2020-6_L2.0-W2.0-P0.65-BL, symbol MothBox_Symbol_Library:JMTV210P02A
- added R39: 10K, MothBox_footprints_Library:R_0603_1608Metric, symbol MothBox_Symbol_Library:R_Small
- added R40, R41: 4.7K, MothBox_footprints_Library:R_0603_1608Metric, symbol MothBox_Symbol_Library:R_Small
Connections:
- net +12V: now also D2.1 (K), Q10.4 (S), Q10.7 (S); no longer J1.3 (Pin_3), J1.4 (Pin_4), U1.4 (Vout+)
- net +24V: now also D4.1 (K); no longer R30.1
- net GND: now also R40.2, R41.1
- net at Q2.3 (D), Q8.3 (G): no longer R30.2
- new net: R39.2, R40.1
- new net: D4.2 (A), R30.2
- new net: D2.2 (A), Q10.3 (G), R39.1
- new net: J1.3 (Pin_3), J1.4 (Pin_4), Q10.1 (D), Q10.2 (D), Q10.5 (D), Q10.6 (D), Q10.8 (D), U1.4 (Vout+)
- new net: R30.1, R41.2
Other:
- note added: "Cut Jumper to measure current flow"
- note added: "Switch the External Regulator on and Off"
- note added: "To External 12V Regulator"
- note removed: "Switch the Regulator on and Off"
- moved on the sheet: J1, Q2, R1, R30, TP5
