File: Hardware/PCB/Andy_PCB_5.0.3/MothBox/MothBox_5.0.3/RPI5.kicad_sch (KiCad schematic)
At the start: 7 parts, among them U4 RASPBERRY_PI_4B_4GB, U5 RASPBERRY_PI_5, U6 RASPBERRY_PI_4B_4GB, U7 Female Inv Socket Pi 2.54-2*20

Commit message: version 5.0.3 completed changes, as per CHANGELOG
Parts:
- removed C1: 1000uF 50V, 0_easyeda_footprints:CAP-TH_BD16.0-P7.50-D1.2-FD, symbol MothBox_Symbol_Library:C_Polarized_Small_US
- added C1, C19, C20, C21: 10uF, MothBox_footprints_Library:C_0603_1608Metric, symbol MothBox_Symbol_Library:C_Small
Connections:
- net +5V: now also C1.1, C19.1, C20.1, C21.1
- net GND: now also C1.2, C19.2, C20.2, C21.2
