File: Hardware/PCB/Andy_PCB_5.0.3/MothBox/UV_LED_PCB.kicad_sch (KiCad schematic)
At the start: 19 parts, among them J4 DB141V-2.54-4P, Q4 YJQ10N2A, Q5 YJQ10N2A, Q6 YJQ10N2A, Q9 YJQ10N2A

Commit message: version 5.0.3 completed changes, as per CHANGELOG
Parts:
- removed D2, D5, D6, D7: ESD12VD3B-TP, MothBox_footprints_Library:D_SOD-323, symbol MothBox_Symbol_Library:ESD5Zxx

Commit message: swapped out Q1, Q8, Q10 for better specc'ed MOSFETs. Moved a few tracks around and updated CHANGELOG.txt
Parts:
- H11, H12, H13: symbol Mechanical:MountingHole -> MothBox_Symbol_Library:MountingHole
Changed lines of the file:
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@@
 	(title_block
 		(title "MothBox")
-		(date "2025-11-05")
+		(date "2025-11-14")
 		(rev "5.0.3")
 		(company "Digital Naturalism Laboritories")
@@
 	)
 	(symbol
-		(lib_id "Mechanical:MountingHole")
+		(lib_id "MothBox_Symbol_Library:MountingHole")
 		(at 227.33 85.09 0)
 		(unit 1)
@@
 	)
 	(symbol
-		(lib_id "Mechanical:MountingHole")
+		(lib_id "MothBox_Symbol_Library:MountingHole")
 		(at 99.06 152.4 0)
 		(unit 1)
@@
 	)
 	(symbol
-		(lib_id "Mechanical:MountingHole")
+		(lib_id "MothBox_Symbol_Library:MountingHole")
 		(at 99.06 85.09 0)
 		(unit 1)
