File: Hardware/PCB/Andy_PCB_5.0.4/MothBox/GPS.kicad_sch (KiCad schematic)
At the start: 22 parts, among them J5 Conn_1.25mm, Q11 AP30P30Q, U10 Days, U11 Hours3, U12 MODE, U13 Hours1, U14 Hours2, U15 PCA9555PW, U16 PCA9555PW, U17 DS18B20U, U18 LTR-303ALS-01, U8 GPs 5 pin PM2.54-1*5, U9 PCA9555PW

Commit message: v5.0.4 schematic and PCB done. Ready for review
Parts:
- removed Q11: AP30P30Q, easyeda2kicad:PDFN3333-8_L3.1-W3.2-P0.65-LS3.4-BL, symbol easyeda2kicad:AP30P30Q
- added Q13: AP30P30Q, MothBox_footprints_Library:PDFN3333-8_L3.1-W3.2-P0.65-LS3.4-BL, symbol MothBox_Symbol_Library:AP30P30Q_1
Connections:
- net +3.3V: now also Q13.5 (D), Q13.6 (D), Q13.7 (D), Q13.8 (D), Q13.9 (D)
- net +3V3: now also Q13.1 (S), Q13.2 (S), Q13.3 (S)
- net 3V3_CTL: now also Q13.4 (G)
Other:
- note added: "From RPi"
- note added: "To Sensors"
- moved on the sheet: R36, TP7
