File: Hardware/PCB/Andy_PCB_5.0.4/MothBox/Power.kicad_sch (KiCad schematic)
At the start: 50 parts, among them J1 DB141V-2.54-4P, J2 DB141V-2.54-4P, J3 DB141V-2.54-4P, Q1 AP30P30Q, Q10 AP30P30Q, Q2 AO3400A, Q8 AP30P30Q, SW2 KH-6X6X5H-STM, U1 Place Holder voltage regulator, U2 XL4015E1, U3 INA219BIDCNT

Commit message: updated schematic 18V Zener from SOD-323 to SOD-123
Parts:
- D1, D2, D4: footprint MothBox_footprints_Library:D_SOD-323 -> Diode_SMD:D_SOD-123
Changed lines of the file:
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@@
 			)
 		)
-		(property "Footprint" "MothBox_footprints_Library:D_SOD-323"
+		(property "Footprint" "Diode_SMD:D_SOD-123"
 			(at 96.52 78.74 90)
 			(effects
@@
 			)
 		)
-		(property "Footprint" "MothBox_footprints_Library:D_SOD-323"
+		(property "Footprint" "Diode_SMD:D_SOD-123"
 			(at 250.19 80.01 90)
 			(effects
@@
 			)
 		)
-		(property "Footprint" "MothBox_footprints_Library:D_SOD-323"
+		(property "Footprint" "Diode_SMD:D_SOD-123"
 			(at 148.59 80.01 90)
 			(effects
